File: lsm6dsv32x_breakout.kicad_pcb (KiCad board)
At the start: 2 copper layers, 20.3 x 7 mm, 9 parts, among them J1 Conn_01x08, U1 LSM6DSV32X

Commit message: Enlarge board to 20.32 x 10.2 mm and add two M2 mounting holes
JLCPCB assembly requires at least 10 x 10 mm. The circuit area moves down
3.2 mm, and the new top band holds two non-plated M2 holes (H1/H2) with a
2 mm copper keepout on both layers. The title and axis marker silkscreen
move into that band.

Also:
- schematic note marks C3 as DNP only when it is in design.DNP
- make_fab.sh aborts if gen_pcb.py fails instead of hiding the error
- README updated for the new size and the mounting holes

Co-Authored-By: Claude Opus 5.5 <noreply@anthropic.com>
Parts:
- added H1: MountingHole_M2, MountingHole:MountingHole_2.2mm_M2, F.Cu at (102.3, 101.9)
- added H2: MountingHole_M2, MountingHole:MountingHole_2.2mm_M2, F.Cu at (118.0, 101.9)
- moved C1 3.20 mm to (114.2, 103.9)
- moved C2 3.20 mm to (108.6, 103.9)
- moved C3 3.20 mm to (106.2, 103.9)
- moved J1 3.20 mm to (101.3, 108.9)
- moved R2 3.20 mm to (104.4, 106.4)
- moved R3 3.20 mm to (116.0, 105.5)
- moved U1 3.20 mm to (111.4, 105.5)
- moved JP1 3.20 mm to (102.2, 106.1)
- moved R1 3.20 mm to (104.4, 107.3)
Other:
- board size 20.3 x 7 mm -> 20.3 x 10.2 mm
