File: lsm6dsv32x_breakout.kicad_sch (KiCad schematic)
At the start: 9 parts, among them J1 Conn_01x08, U1 LSM6DSV32X

Commit message: Enlarge board to 20.32 x 10.2 mm and add two M2 mounting holes
JLCPCB assembly requires at least 10 x 10 mm. The circuit area moves down
3.2 mm, and the new top band holds two non-plated M2 holes (H1/H2) with a
2 mm copper keepout on both layers. The title and axis marker silkscreen
move into that band.

Also:
- schematic note marks C3 as DNP only when it is in design.DNP
- make_fab.sh aborts if gen_pcb.py fails instead of hiding the error
- README updated for the new size and the mounting holes

Co-Authored-By: Claude Opus 5.5 <noreply@anthropic.com>
Parts:
- added H1, H2: MountingHole_M2, MountingHole:MountingHole_2.2mm_M2, symbol Mechanical:MountingHole
Changed lines of the file:
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@@
+	)
+	(symbol
+		(lib_id "Mechanical:MountingHole")
+		(at 203.2 91.44 0)
+		(unit 1)
+		(exclude_from_sim no)
+		(in_bom no)
+		(on_board yes)
+		(dnp no)
+		(fields_autoplaced yes)
+		(property "Reference" "H1"
+			(at 203.2 86.36 0)
+			(effects
+				(font
+					(size 1.27 1.27)
+				)
+			)
+		)
+		(property "Value" "MountingHole_M2"
+			(at 203.2 88.265 0)
+			(effects
+				(font
+					(size 1.27 1.27)
+				)
+			)
+		)
+		(property "Footprint" "MountingHole:MountingHole_2.2mm_M2"
+			(at 203.2 91.44 0)
+			(effects
+				(font
+					(size 1.27 1.27)
+				)
+				(hide yes)
+			)
+		)
+		(property "Datasheet" "~"
+			(at 203.2 91.44 0)
+			(effects
+				(font
+					(size 1.27 1.27)
+				)
+				(hide yes)
+			)
+		)
+		(property "Description" "Mounting Hole without connection"
+			(at 203.2 91.44 0)
+			(effects
+				(font
+					(size 1.27 1.27)
+				)
+				(hide yes)
+			)
+		)
+		(instances
+			(project "lsm6dsv32x_breakout"
+				(path "/0c73b162-4912-506b-b411-aeeb1302e4c7"
+					(reference "H1")
+					(unit 1)
+				)
+			)
+		)
+	)
+	(symbol
+		(lib_id "Mechanical:MountingHole")
+		(at 213.36 91.44 0)
+		(unit 1)
+		(exclude_from_sim no)
+		(in_bom no)
+		(on_board yes)
+		(dnp no)
+		(fields_autoplaced yes)
+		(property "Reference" "H2"
+			(at 213.36 86.36 0)
+			(effects
+				(font
+					(size 1.27 1.27)
+				)
+			)
+		)
+		(property "Value" "MountingHole_M2"
+			(at 213.36 88.265 0)
+			(effects
+				(font
+					(size 1.27 1.27)
+				)
+			)
+		)
+		(property "Footprint" "MountingHole:MountingHole_2.2mm_M2"
+			(at 213.36 91.44 0)
+			(effects
+				(font
+					(size 1.27 1.27)
+				)
+				(hide yes)
+			)
+		)
+		(property "Datasheet" "~"
+			(at 213.36 91.44 0)
+			(effects
+				(font
+					(size 1.27 1.27)
+				)
+				(hide yes)
+			)
+		)
+		(property "Description" "Mounting Hole without connection"
+			(at 213.36 91.44 0)
+			(effects
+				(font
+					(size 1.27 1.27)
+				)
+				(hide yes)
+			)
+		)
+		(instances
+			(project "lsm6dsv32x_breakout"
+				(path "/0c73b162-4912-506b-b411-aeeb1302e4c7"
+					(reference "H2")
+					(unit 1)
+				)
+			)
+		)
 	)
 	(symbol
@@
 		)
 	)
-	(text "Notes:\n- 3.3 V only: VDD and VDDIO are tied together (no regulator / level shifter).\n- I2C address 0x6B: SA0 pulled up by R3. Drive SDO low from the header for 0x6A.\n- CS has an internal pull-up, so the part starts in I2C/I3C mode; pull CS low for SPI.\n- JP1 (bridged by default) enables the 10k SCL/SDA pull-ups. Cut it to remove them.\n- SDx/SCx tied to GND (analog hub / Qvar / sensor hub not used), OCS_Aux/SDO_Aux left open\n  per datasheet Table 2 / Figure 28.\n- C3 (4.7uF) is DNP: optional bulk capacitor for noisy or long 3.3 V wiring."
+	(text "Notes:\n- 3.3 V only: VDD and VDDIO are tied together (no regulator / level shifter).\n- I2C address 0x6B: SA0 pulled up by R3. Drive SDO low from the header for 0x6A.\n- CS has an internal pull-up, so the part starts in I2C/I3C mode; pull CS low for SPI.\n- JP1 (bridged by default) enables the 10k SCL/SDA pull-ups. Cut it to remove them.\n- SDx/SCx tied to GND (analog hub / Qvar / sensor hub not used), OCS_Aux/SDO_Aux left open\n  per datasheet Table 2 / Figure 28.\n- C3 (4.7uF): optional bulk capacitor for noisy or long 3.3 V wiring."
 		(exclude_from_sim no)
 		(at 76.2 162.56 0)
